File: embebeed.kicad_sch (KiCad schematic)
At the start: 30 parts

Commit message: Adicionado os diodos no motor e buzzer
Parts:
- added D (x2): DIODE, symbol pspice:DIODE
- gave numbers to parts that had none: 2
Connections:
- net GND: now also BUZZER_OPTO.4, MOTOROPTo.4; no longer Ventoinha.2 (-), alarme.2 (+)
- net VDD_5v: now also 200ohm.1; no longer 200ohm.2
- net at alarme.1 (-): now also 200ohm.1, D.2 (A); no longer BUZZER_OPTO.4
- net at BUZZER_OPTO.5: now also alarme.2 (+), D.1 (K); no longer 200ohm.1
- net at Ventoinha.1 (+): now also 200ohm.2, D.2 (A); no longer MOTOROPTo.4
- net at MOTOROPTo.5: now also Ventoinha.2 (-), D.1 (K); no longer 200ohm.1
Other:
- moved on the sheet: 200ohm, 300ohms, BUZZER_OPTO, MOTOROPTo, TIVA_to_can_transciver, Ventoinha, alarme
