File: embebeed.kicad_sch (KiCad schematic)
At the start: 29 parts

Commit message: Teste de interrupt com keypad para o Tiva C
Connections:
- net ENABLE: no longer DISPLAY_LCD.P$6
- net PB2: no longer 10k.2, DISPLAY_LCD.P$7
- net PD6: no longer DISPLAY_LCD.P$12
- net PD7: no longer DISPLAY_LCD.P$13
- net PF4: now also DISPLAY_LCD.P$11; no longer DISPLAY_LCD.P$14, teclas. (Y4)
- net RS: now also TIVA.J4_2 (PF3); no longer DISPLAY_LCD.P$4
- net SPI_CLOCK: no longer TIVA.J2_10 (PA2)
- net SPI_INPUT: no longer TIVA.J2_8 (PA4)
- net SPI_OUTPUT: no longer TIVA.J1_8 (PA5)
- net SPI_SS: now reaches TIVA.J1_2 (PB5)
- net CAN_RX: now reaches TIVA.J1_5 (PE4)
- net CAN_TX: now reaches TIVA.J1_6 (PE5)
- net SPI_Clock: now reaches TIVA.J1_7 (PB4)
- net Y4: now reaches TIVA.J2_2 (PB2)
- net MOSI: now reaches TIVA.J2_6 (PB7)
- net MISO: now reaches TIVA.J2_7 (PB6)
- net DB6: now reaches TIVA.J2_9 (PA3)
- net EN: now reaches TIVA.J4_1 (PF2)
- net DB4: now reaches TIVA.J4_10 (PF4)
- net Y1: now reaches TIVA.J4_3 (PB3)
- net X2: now reaches TIVA.J4_4 (PC4)
- net X3: now reaches TIVA.J4_5 (PC5)
- net X4: now reaches TIVA.J4_6 (PC6)
- net X1: now reaches TIVA.J4_7 (PC7)
- net Y2: now reaches TIVA.J4_8 (PD6)
- net Y3: now reaches TIVA.J4_9 (PD7)
- removed net PB6: DISPLAY_LCD.P$11, teclas. (Y4)
- removed net PB7: 10k.2, DISPLAY_LCD.P$10, teclas. (Y4)
- removed net PE0: 10k.2, DISPLAY_LCD.P$8, teclas. (Y4)
- removed net PF0: 10k.2, DISPLAY_LCD.P$9, teclas. (Y4)
- new net DB5: TIVA.J2_10 (PA2)
- new net DB7: TIVA.J2_8 (PA4)
- new net PA2: DISPLAY_LCD.P$12
- new net PA3: DISPLAY_LCD.P$13
- new net PA4: DISPLAY_LCD.P$14
- new net PB3: teclas. (Y4)
- new net PC4: 10k.2, teclas. (Y4)
- new net PC5: 10k.2, teclas. (Y4)
- new net PC6: 10k.2, teclas. (Y4)
- new net PC7: 10k.2, teclas. (Y4)
- new net PF2: DISPLAY_LCD.P$6
- new net PF3: DISPLAY_LCD.P$4
