File: embebeed.kicad_sch (KiCad schematic)
At the start: 29 parts

Commit message: teste do LCD
Connections:
- net DB4: now also TIVA.J1_8 (PA5)
- net PF4 renamed PA5
Changed lines of the file:
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@@
     (effects (font (size 1.27 1.27)) (justify left bottom))
   )
-  (label "PF4" (at 24.13 165.1 0)
+  (label "PA5" (at 24.13 165.1 0)
     (effects (font (size 1.27 1.27)) (justify left bottom))
   )
@@
     (effects (font (size 1.27 1.27)) (justify left bottom))
   )
+  (label "DB4" (at 53.34 54.61 0)
+    (effects (font (size 1.27 1.27)) (justify left bottom))
+  )

Commit message: Havia esquecido de upa o keypad+LCD
Connections:
- net DB4: no longer TIVA.J4_10 (PF4)
- net RS: no longer TIVA.J3_3 (PD0)
- new net Não usar: TIVA.J3_3 (PD0)
Changed lines of the file:
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@@
-    (effects (font (size 1.27 1.27)) (justify left bottom))
-  )
-  (label "DB4" (at 99.06 92.71 0)
     (effects (font (size 1.27 1.27)) (justify left bottom))
   )
@@
     (effects (font (size 1.27 1.27)) (justify left bottom))
   )
-  (label "RS" (at 104.14 64.77 0)
-    (effects (font (size 1.27 1.27)) (justify left bottom))
-  )
+  (label "Não usar" (at 104.14 64.77 0)
+    (effects (font (size 1.27 1.27)) (justify left bottom))
+  )
